File: Kicad Workspace/mcu.kicad_sch (KiCad schematic)
At the start: 2 parts, among them U9 STM32G030C8Tx

Commit message: feat: schematics almost done, starting to correct compile pb
Parts:
- removed RV1: R_Potentiometer, symbol Device:R_Potentiometer
Connections:
- net MUX_SEL: now reaches U9.22 (MUX_SEL)
- net MUTE_DAC: now reaches U9.23 (MUTE_DAC)
- net RESET_BT: now reaches U9.24 (RESET_BT)
- net RESET_AMP: now reaches U9.25 (RESET_AMP)
- net FAULT_AMP: now reaches U9.26 (FAULT_AMP)
- net TX: now reaches U9.29 (USART1_TX)
- net RX: now reaches U9.32 (USART1_RX)
- net CTS: now reaches U9.33 (USART1_CTS)
- net RTS: now reaches U9.34 (USART1_RTS)
- net SCL: now reaches U9.45 (I2C_SCL)
- net SDA: now reaches U9.46 (I2C_SDA)

Commit message: fix: Bus fix with correct syntax
Connections:
- net CTS renamed UART.CTS
- net RTS renamed UART.RTS
- net RX renamed UART.RX
- net SCL renamed I2C.SCL
- net SDA renamed I2C.SDA
- net TX renamed UART.TX
Changed lines of the file:
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@@
 		)
 	)
-	(label "SCL"
+	(label "I2C.SCL"
 		(at 167.64 116.84 0)
 		(effects
@@
 		)
 	)
-	(label "RTS"
+	(label "UART.RTS"
 		(at 163.83 90.17 0)
 		(effects
@@
 		)
 	)
-	(label "SDA"
+	(label "I2C.SDA"
 		(at 167.64 119.38 0)
 		(effects
@@
 		)
 	)
-	(label "RX"
+	(label "UART.RX"
 		(at 163.8089 85.09 0)
 		(effects
@@
 		)
 	)
-	(label "CTS"
+	(label "UART.CTS"
 		(at 163.83 87.63 0)
 		(effects
@@
 		)
 	)
-	(label "TX"
+	(label "UART.TX"
 		(at 163.8089 82.55 0)
 		(effects

Commit message: feat: potentiometers + source switch + bt pari button
Parts:
- added J10, J11, J12, J13, J9: Conn_01x03_Pin, Connector_PinHeader_2.54mm:PinHeader_1x03_P2.54mm_Vertical, symbol Connector:Conn_01x03_Pin
- added R38, R39, R40: 2.2K, Resistor_SMD:R_0201_0603Metric, symbol Device:R
- added SW1: SW_Rotary_1x4_MP, symbol Switch:SW_Rotary_1x4_MP
- added SW2: (no value), Button_Switch_THT:SW_PUSH_6mm, symbol Switch:SW_Push
Connections:
- net GND: now also J10.3 (Pin_3), J11.3 (Pin_3), J12.3 (Pin_3), J13.3 (Pin_3), J9.3 (Pin_3), R40.2, SW1.4, SW1.MP, SW2.2
- net at U9.11 (Volume): now also J9.2 (Pin_2)
- net at U9.12 (L/R): now also J10.2 (Pin_2)
- net at U9.13 (EQ_low): now also J11.2 (Pin_2)
- net at U9.14 (EQ_midle): now also J12.2 (Pin_2)
- net at U9.15 (EQ_high): now also J13.2 (Pin_2)
- net at U9.16 (Source): now also SW1.5
- net at U9.48 (PAIR_BT): now also SW2.1
- new net: R38.1, R39.2, SW1.2
- new net: R38.2, R40.1, SW1.3
- new net +3.3VA: J10.1 (Pin_1), J11.1 (Pin_1), J12.1 (Pin_1), J13.1 (Pin_1), J9.1 (Pin_1), R39.1, SW1.1
