File: Kicad Workspace/mcu.kicad_sch (KiCad schematic)
At the start: 11 parts, among them J10 Conn_01x03_Pin, J11 Conn_01x03_Pin, J12 Conn_01x03_Pin, J13 Conn_01x03_Pin, J9 Conn_01x03_Pin, SW1 SW_Rotary_1x4_MP, U9 STM32G030C8Tx

Commit message: fix: schematic corrections from the datasheet audit
Eight defects found by checking every pin of the six sheets against the
datasheets in Ressources/Datasheet.

MCU sheet:
- add R37/R41 (2.2K) I2C pull-ups on SDA/SCL, sized for the 400 kHz bus
- add R42 (2.2K) pull-up on PAIR_BT, SW2 had no defined idle level
- add C82/C83/C84 decoupling on the STM32 supply pins
- tie VREF+ to +3.3V, it was left unconnected so the ADC had no reference
- move the potentiometers and SW1 from +3.3VA to +3.3V, the analog rail is
  reserved for the audio path and the readings are ratiometric anyway

Amplification sheet:
- add C85 (10uF/25V) and C86 (0.1uF/16V) on the TPA3255 VDD, the 12V
  housekeeping rail had no local decoupling
Parts:
- added C82, C84: 0.1µF/16V, Capacitor_SMD:C_0402_1005Metric, symbol Device:C
- added C83: 10µF/25V, Capacitor_SMD:C_0805_2012Metric, symbol Device:C
- added R37, R41, R42: 2.2K, Resistor_SMD:R_0201_0603Metric, symbol Device:R
Connections:
- net +3.3VA is gone; now on net +3.3V: J10.1 (Pin_1), J11.1 (Pin_1), J12.1 (Pin_1), J13.1 (Pin_1), J9.1 (Pin_1), R39.1, SW1.1
- net +3.3V: now also U9.5 (VREF+), C82.1, C83.1, C84.2, R37.2, R41.1, R42.2
- net GND: now also C82.2, C83.2, C84.1
- net I2C.SCL: now also R37.1
- net I2C.SDA: now also R41.2
- net at SW2.1, U9.48 (PAIR_BT): now also R42.1
Other:
- moved on the sheet: SW2
