File: Kicad Workspace/Kicad Workspace.kicad_sch (KiCad schematic)
At the start: 0 parts

Commit message: fix: Bus fix with correct syntax
Other:
- sheet Amplification ports: added none; removed L+, L-, R+, R-
- sheet Bluetooth ports: added BT_I2S{DATA BCK LRCK}; removed BT_I2S{BT_BCK BT_DATA BT_LRCK}
- sheet EQ and DAC ports: added BT_I2S{DATA BCK LRCK}, WIRE_I2S{DATA BCK LRCK}; removed BT_I2S{BT_DATA BT_BCK BT_LRCK}, WIRE_I2S{WIRE_DATA WIRE_BCK WIRE_LRCK}
- sheet Wired Input ports: added I2C{SCL SDA}, WIRE_I2S{DATA BCK LRCK}; removed AUX, LINE, MONO, WIRE_I2S{WIRE_DATA WIRE_BCK WIRE_LRCK}
Changed lines of the file:
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@@
 			)
 		)
-		(pin "WIRE_I2S{WIRE_DATA WIRE_BCK WIRE_LRCK}" output
+		(pin "I2C{SCL SDA}" bidirectional
+			(at 71.12 52.07 270)
+			(effects
+				(font
+					(size 1.27 1.27)
+				)
+				(justify left)
+			)
+		)
+		(pin "WIRE_I2S{DATA BCK LRCK}" output
 			(at 80.01 27.94 0)
 			(effects
@@
 				)
 				(justify right)
-			)
-		)
-		(pin "MONO" input
-			(at 19.05 31.75 180)
-			(effects
-				(font
-					(size 1.27 1.27)
-				)
-				(justify left)
-			)
-		)
-		(pin "AUX" input
-			(at 19.05 35.56 180)
-			(effects
-				(font
-					(size 1.27 1.27)
-				)
-				(justify left)
-			)
-		)
-		(pin "LINE" input
-			(at 19.05 39.37 180)
-			(effects
-				(font
-					(size 1.27 1.27)
-				)
-				(justify left)
 			)
 		)
@@
 			)
 		)
-		(pin "BT_I2S{BT_DATA BT_BCK BT_LRCK}" input
-			(at 97.79 31.75 180)
-			(effects
-				(font
-					(size 1.27 1.27)
-				)
-				(justify left)
-			)
-		)
-		(pin "WIRE_I2S{WIRE_DATA WIRE_BCK WIRE_LRCK}" input
-			(at 97.79 27.94 180)
-			(effects
-				(font
-					(size 1.27 1.27)
-				)
-				(justify left)
-			)
-		)
 		(pin "I2C{SCL SDA}" bidirectional
 			(at 123.19 48.26 270)
+			(effects
+				(font
+					(size 1.27 1.27)
+				)
+				(justify left)
+			)
+		)
+		(pin "BT_I2S{DATA BCK LRCK}" input
+			(at 97.79 31.75 180)
+			(effects
+				(font
+					(size 1.27 1.27)
+				)
+				(justify left)
+			)
+		)
+		(pin "WIRE_I2S{DATA BCK LRCK}" input
+			(at 97.79 27.94 180)
 			(effects
 				(font
@@
 			)
 		)
-		(pin "BT_I2S{BT_BCK BT_DATA BT_LRCK}" output
+		(pin "BT_I2S{DATA BCK LRCK}" output
 			(at 78.74 76.2 0)
 			(effects
@@
 			)
 		)
-		(pin "L+" output
-			(at 205.74 35.56 0)
-			(effects
-				(font
-					(size 1.27 1.27)
-				)
-				(justify right)
-			)
-		)
-		(pin "L-" output
-			(at 205.74 38.1 0)
-			(effects
-				(font
-					(size 1.27 1.27)
-				)
-				(justify right)
-			)
-		)
-		(pin "R+" output
-			(at 205.74 43.18 0)
-			(effects
-				(font
-					(size 1.27 1.27)
-				)
-				(justify right)
-			)
-		)
-		(pin "R-" output
-			(at 205.74 45.72 0)
-			(effects
-				(font
-					(size 1.27 1.27)
-				)
-				(justify right)
-			)
-		)
