File: Kicad Workspace/bluetooth.kicad_sch (KiCad schematic)
At the start: 7 parts

Commit message: feat: schematics almost done, starting to correct compile pb
Connections:
- net TX: now reaches U1.13 (BT_TX/PIO5)
- net RX: now reaches U1.14 (BT_RX/PIO4)
- net CTS: now reaches U1.15 (BT_CTS/PIO3)
- net RTS: now reaches U1.16 (BT_RTS/PIO2)
- net BT_BCK: now reaches U1.4 (PCM_CLK/PIO16)
- net BT_DATA: now reaches U1.6 (PCM_OUT/PIO18)
- net BT_LRCK: now reaches U1.7 (PCM_SYNC/PIO17)
- no-connect marks 34 -> 35
Changed lines of the file:
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@@
+	)
+	(no_connect
+		(at 95.25 85.09)
 	)
 	(no_connect
@@
 	)
 	(bus_entry
-		(at 55.88 85.09)
-		(size -2.54 -2.54)
-		(stroke
-			(width 0)
-			(type default)
-		)
-	)
-	(bus_entry
 		(at 76.2 111.76)
 		(size -2.54 -2.54)
@@
 	(wire
 		(pts
-			(xy 55.88 85.09) (xy 95.25 85.09)
-		)
-		(stroke
-			(width 0)
-			(type default)
-		)
-	)
-	(wire
-		(pts
 			(xy 186.69 134.62) (xy 195.58 134.62)
 		)
@@
 		)
 	)
+	(wire
+		(pts
+			(xy 179.07 54.61) (xy 185.42 54.61)
+		)
+		(stroke
+			(width 0)
+			(type default)
+		)
+	)
+	(wire
+		(pts
+			(xy 76.2 100.33) (xy 95.25 100.33)
+		)
+		(stroke
+			(width 0)
+			(type default)
+		)
+	)
+	(wire
+		(pts
+			(xy 55.88 77.47) (xy 95.25 77.47)
+		)
+		(stroke
+			(width 0)
+			(type default)
+		)
+	)
 	(bus
 		(pts
-			(xy 53.34 60.96) (xy 53.34 82.55)
-		)
-		(stroke
-			(width 0)
-			(type default)
-		)
-	)
-	(wire
-		(pts
-			(xy 179.07 54.61) (xy 185.42 54.61)
-		)
-		(stroke
-			(width 0)
-			(type default)
-		)
-	)
-	(wire
-		(pts
-			(xy 76.2 100.33) (xy 95.25 100.33)
-		)
-		(stroke
-			(width 0)
-			(type default)
-		)
-	)
-	(wire
-		(pts
-			(xy 55.88 77.47) (xy 95.25 77.47)
+			(xy 53.34 60.96) (xy 53.34 74.93)
 		)
 		(stroke
@@
 		)
 	)
-	(hierarchical_label "BT_UART"
-		(shape input)
+	(label "BT_DATA"
+		(at 59.69 73.66 0)
+		(effects
+			(font
+				(size 1.27 1.27)
+			)
+			(justify left bottom)
+		)
+	)
+	(label "RX"
+		(at 80.01 104.14 0)
+		(effects
+			(font
+				(size 1.27 1.27)
+			)
+			(justify left bottom)
+		)
+	)
+	(label "RTS"
+		(at 79.66 111.76 0)
+		(effects
+			(font
+				(size 1.27 1.27)
+			)
+			(justify left bottom)
+		)
+	)
+	(label "BT_BCK"
+		(at 59.69 66.04 0)
+		(effects
+			(font
+				(size 1.27 1.27)
+			)
+			(justify left bottom)
+		)
+	)
+	(label "TX"
+		(at 80.01 100.33 0)
+		(effects
+			(font
+				(size 1.27 1.27)
+			)
+			(justify left bottom)
+		)
+	)
+	(label "CTS"
+		(at 79.8254 107.95 0)
+		(effects
+			(font
+				(size 1.27 1.27)
+			)
+			(justify left bottom)
+		)
+	)
+	(label "BT_LRCK"
+		(at 59.69 77.47 0)
+		(effects
+			(font
+				(size 1.27 1.27)
+			)
+			(justify left bottom)
+		)
+	)
+	(hierarchical_label "UART{TX RX CTS RTS}"
+		(shape bidirectional)
 		(at 73.66 95.25 180)
 		(effects
@@
 		)
 	)
-	(hierarchical_label "BT_I2S"
+	(hierarchical_label "BT_I2S{BT_BCK BT_DATA BT_LRCK}"
 		(shape output)
 		(at 53.34 60.96 180)

Commit message: feat: correction work in progress
Connections:
- net CTS: no longer names the net of U1.15 (BT_CTS/PIO3)
- net RTS: no longer names the net of U1.16 (BT_RTS/PIO2)
- net RX: no longer names the net of U1.14 (BT_RX/PIO4)
- net TX: no longer names the net of U1.13 (BT_TX/PIO5)
Changed lines of the file:
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@@
-		)
-	)
-	(label "RX"
-		(at 80.01 104.14 0)
-		(effects
-			(font
-				(size 1.27 1.27)
-			)
-			(justify left bottom)
-		)
-	)
-	(label "RTS"
-		(at 79.66 111.76 0)
-		(effects
-			(font
-				(size 1.27 1.27)
-			)
-			(justify left bottom)
 		)
 	)
@@
 		(effects
 			(font
-				(size 1.27 1.27)
-			)
-			(justify left bottom)
-		)
-	)
-	(label "TX"
-		(at 80.01 100.33 0)
-		(effects
-			(font
-				(size 1.27 1.27)
-			)
-			(justify left bottom)
-		)
-	)
-	(label "CTS"
-		(at 79.8254 107.95 0)
-		(effects
-			(font

Commit message: feat: BT-1058 footprint name update
Parts:
- U1: footprint (none) -> FootPrints:FSC-BT1058
Changed lines of the file:
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@@
 			)
 		)
-		(property "Footprint" ""
+		(property "Footprint" "FootPrints:FSC-BT1058"
 			(at 101.6 67.31 0)
 			(hide yes)

Commit message: fix: Bus fix with correct syntax
Parts:
- R11: footprint Resistor_SMD:R_01005_0402Metric -> Resistor_SMD:R_0201_0603Metric
Connections:
- net UART.RX: now reaches U1.13 (BT_TX/PIO5)
- net UART.TX: now reaches U1.14 (BT_RX/PIO4)
- net UART.RTS: now reaches U1.15 (BT_CTS/PIO3)
- net UART.CTS: now reaches U1.16 (BT_RTS/PIO2)
- net BT_BCK renamed BT_I2S.BCK
- net BT_DATA renamed BT_I2S.DATA
- net BT_LRCK renamed BT_I2S.LRCK
Changed lines of the file:
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@@
 		)
 	)
-	(label "BT_DATA"
+	(label "BT_I2S.DATA"
 		(at 59.69 73.66 0)
 		(effects
@@
 		)
 	)
-	(label "BT_BCK"
+	(label "UART.RX"
+		(at 76.2 100.33 0)
+		(effects
+			(font
+				(size 1.27 1.27)
+			)
+			(justify left bottom)
+		)
+	)
+	(label "BT_I2S.BCK"
 		(at 59.69 66.04 0)
 		(effects
@@
 		)
 	)
-	(label "BT_LRCK"
+	(label "UART.RTS"
+		(at 76.2 107.95 0)
+		(effects
+			(font
+				(size 1.27 1.27)
+			)
+			(justify left bottom)
+		)
+	)
+	(label "UART.CTS"
+		(at 76.2 111.76 0)
+		(effects
+			(font
+				(size 1.27 1.27)
+			)
+			(justify left bottom)
+		)
+	)
+	(label "BT_I2S.LRCK"
 		(at 59.69 77.47 0)
+		(effects
+			(font
+				(size 1.27 1.27)
+			)
+			(justify left bottom)
+		)
+	)
+	(label "UART.TX"
+		(at 76.2 104.14 0)
 		(effects
 			(font
@@
 		)
 	)
-	(hierarchical_label "BT_I2S{BT_BCK BT_DATA BT_LRCK}"
+	(hierarchical_label "BT_I2S{DATA BCK LRCK}"
 		(shape output)
 		(at 53.34 60.96 180)
@@
 			)
 		)
-		(property "Footprint" "Resistor_SMD:R_01005_0402Metric"
+		(property "Footprint" "Resistor_SMD:R_0201_0603Metric"
 			(at 182.88 124.968 90)
 			(hide yes)
