File: Kicad Workspace/bluetooth.kicad_sch (KiCad schematic)
At the start: 7 parts

Commit message: feat: kicad alim stage clean up + TPA stage clean up
Parts:
- R11: footprint Resistor_SMD:R_0201_0603Metric -> Resistor_SMD:R_0402_1005Metric
Changed lines of the file:
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@@
 			)
 		)
-		(property "Footprint" "Resistor_SMD:R_0201_0603Metric"
+		(property "Footprint" "Resistor_SMD:R_0402_1005Metric"
 			(at 182.88 124.968 90)
 			(hide yes)
