File: Kicad Workspace/eq_and_dac.kicad_sch (KiCad schematic)
At the start: 22 parts, among them U3 PCM5242RHBT, U4 TMUX1574PW

Commit message: feat: routing work in progress
Parts:
- U3: footprint PCM5242RHBT:IC_ADS125H01IRHBT -> FootPrints:PCM5242
Changed lines of the file:
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@@
 			)
 		)
-		(property "Footprint" "PCM5242RHBT:IC_ADS125H01IRHBT"
+		(property "Footprint" "FootPrints:PCM5242"
 			(at 185.42 102.87 0)
 			(hide yes)
