File: Kicad Workspace/eq_and_dac.kicad_sch (KiCad schematic)
At the start: 22 parts, among them U3 PCM5242RHBT, U4 TMUX1574PW

Commit message: feat: routing work in progress
Parts:
- C5: footprint Capacitor_SMD:C_0805_2012Metric -> Capacitor_SMD:C_0201_0603Metric
Changed lines of the file:
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@@
 			)
 		)
-		(property "Footprint" "Capacitor_SMD:C_0805_2012Metric"
+		(property "Footprint" "Capacitor_SMD:C_0201_0603Metric"
 			(at 223.2152 72.39 0)
 			(hide yes)
