File: Kicad Workspace/Kicad Workspace.kicad_pcb (KiCad board)
At the start: 2 copper layers, 141 parts, among them J1 NMJ4HFD2, J10 Conn_01x03_Pin, J11 Conn_01x03_Pin, J12 Conn_01x03_Pin, J13 Conn_01x03_Pin, J2 NMJ4HFD2, J3 AudioJack3_Switch, J4 NMJ4HFD2, J5 L+, J6 L-, J7 R+, J8 R-, J9 Conn_01x03_Pin, U2 PCM1863DBT, U3 PCM5242RHBT, U4 TMUX1574PW, U5 TPA3255DDV, U6 TLV76733DRVx, U7 LM5017MR, U8 LT3042xMSE, U9 STM32G030C8Tx, Y1 Crystal

Commit message: feat: kicad alim stage clean up + TPA stage clean up
Parts:
- added C60: 10µF/50V, Capacitor_THT:CP_Radial_D6.3mm_P2.50mm, F.Cu at (273.2, 136.5)
- added C61: 10µF/50V, Capacitor_THT:CP_Radial_D6.3mm_P2.50mm, F.Cu at (273.2, 144.3)
- added C62: 10µF/50V, Capacitor_THT:CP_Radial_D6.3mm_P2.50mm, F.Cu at (273.2, 152.2)
- added C75: 4.7µF/100V, Capacitor_SMD:C_1210_3225Metric, F.Cu at (287.7, 148.7)
- added C76: 100nF/100V, Capacitor_SMD:C_0805_2012Metric, F.Cu at (296.8, 148.1)
- added C77: 1µF/25V, Capacitor_SMD:C_0805_2012Metric, F.Cu at (296.8, 151.1)
- added C78: 10nF/50V, Capacitor_SMD:C_0603_1608Metric, F.Cu at (292.5, 147.8)
- added C79: 3.3nF/50V, Capacitor_SMD:C_0603_1608Metric, F.Cu at (292.5, 150.4)
- added C80: 100nF/50V, Capacitor_SMD:C_0603_1608Metric, F.Cu at (292.5, 152.9)
- added C81: 22µF/25V, Capacitor_SMD:C_1210_3225Metric, F.Cu at (287.7, 153.0)
- added C82: 0.1µF/16V, Capacitor_SMD:C_0402_1005Metric, F.Cu at (288.8, 162.6)
- added C83: 10µF/25V, Capacitor_SMD:C_0805_2012Metric, F.Cu at (289.5, 160.1)
- added C84: 0.1µF/16V, Capacitor_SMD:C_0402_1005Metric, F.Cu at (288.8, 164.6)
- added C85: 10µF/25V, Capacitor_SMD:C_0805_2012Metric, F.Cu at (280.6, 134.1)
- added C86: 0.1µF/16V, Capacitor_SMD:C_0402_1005Metric, F.Cu at (279.9, 136.5)
- added C87: 10µF/50V, Capacitor_THT:CP_Radial_D6.3mm_P2.50mm, F.Cu at (273.2, 160.0)
- added C88: 4.7µF/25V, Capacitor_SMD:C_0603_1608Metric, F.Cu at (292.5, 155.4)
- added L5: 100µH, Inductor_SMD:L_Bourns_SRR1260, F.Cu at (291.9, 139.6)
- added R37: 2.2K, Resistor_SMD:R_0201_0603Metric, F.Cu at (286.1, 159.5)
- added R41: 2.2K, Resistor_SMD:R_0201_0603Metric, F.Cu at (286.1, 161.3)
- added R42: 2.2K, Resistor_SMD:R_0201_0603Metric, F.Cu at (286.1, 163.0)
- C33, C38, C39: value 1µF -> 1µF/25V; footprint Capacitor_SMD:C_0201_0603Metric -> Capacitor_SMD:C_0603_1608Metric
- C41, C42: footprint Capacitor_SMD:C_01005_0402Metric -> Capacitor_SMD:C_0603_1608Metric
- C43: value 33nF -> 33nF / 50V; footprint Capacitor_SMD:C_0201_0603Metric -> Capacitor_SMD:C_0603_1608Metric
- C44, C45, C46: value 33nF -> 33nF/50V; footprint Capacitor_SMD:C_0201_0603Metric -> Capacitor_SMD:C_0603_1608Metric
- C63, C64, C67, C68: footprint Capacitor_THT:C_Rect_L10.0mm_W4.0mm_P7.50mm_MKS4 -> Capacitor_SMD:C_1206_3216Metric
- C74: value 2.2µF -> 2.2µF/25V; footprint Capacitor_SMD:C_0201_0603Metric -> Capacitor_SMD:C_0603_1608Metric
- R11: footprint Resistor_SMD:R_0201_0603Metric -> Resistor_SMD:R_0402_1005Metric
- R31, R32, R33, R35, R36: footprint Resistor_SMD:R_01005_0402Metric -> Resistor_SMD:R_0603_1608Metric
- R34: value 51.1K -> 100K; footprint Resistor_SMD:R_0201_0603Metric -> Resistor_SMD:R_0603_1608Metric
- moved C71 43.5 mm to (299.9, 202.1)
- moved C72 43.5 mm to (299.9, 205.1)
- moved C73 43.5 mm to (299.9, 208.1)
- moved R31 43.5 mm to (303.2, 201.4)
- moved C74 43.5 mm to (305.6, 201.5)
- moved R21 43.5 mm to (305.6, 203.2)
- moved R30 43.5 mm to (306.5, 207.3)
- moved R32 43.5 mm to (303.2, 203.1)
- moved R33 43.5 mm to (303.2, 204.7)
- moved R34 43.5 mm to (305.6, 205.0)
- moved R35 43.5 mm to (303.2, 206.4)
- moved R36 43.5 mm to (303.2, 208.0)
- moved U6 24.8 mm to (272.5, 182.7)
- moved U7 24.8 mm to (267.6, 177.6)
- moved U8 24.8 mm to (267.0, 183.1)
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Connections:
- J10 pad 1: +3.3VA -> +3.3V
- J11 pad 1: +3.3VA -> +3.3V
- J12 pad 1: +3.3VA -> +3.3V
- J13 pad 1: +3.3VA -> +3.3V
- J9 pad 1: +3.3VA -> +3.3V
- R39 pad 1: +3.3VA -> +3.3V
- U9 pad 5: unconnected-(U9-VREF+-Pad5) -> +3.3V
Routing:
- net +3.3V: track 13.0 -> 14.1 mm
