File: Kicad Workspace/alimentation.kicad_sch (KiCad schematic)
At the start: 23 parts, among them U6 TLV76733DRVx, U7 LM5017MR, U8 LT3042xMSE

Commit message: feat: kicad alim stage clean up + TPA stage clean up
Parts:
- removed C75: 4.7µF, symbol Device:C_Polarized_US
- removed C76: 0.1µF, symbol Device:C_Polarized_US
- removed C77: 1µF, symbol Device:C_Polarized_US
- removed C78: 0.01µF, symbol Device:C_Polarized_US
- removed C81: 22µF, symbol Device:C_Polarized_US
- added C75: 4.7µF/100V, Capacitor_SMD:C_1210_3225Metric, symbol Device:C
- added C76: 100nF/100V, Capacitor_SMD:C_0805_2012Metric, symbol Device:C
- added C77: 1µF/25V, Capacitor_SMD:C_0805_2012Metric, symbol Device:C
- added C78: 10nF/50V, Capacitor_SMD:C_0603_1608Metric, symbol Device:C
- added C81: 22µF/25V, Capacitor_SMD:C_1210_3225Metric, symbol Device:C
- added C88: 4.7µF/25V, Capacitor_SMD:C_0603_1608Metric, symbol Device:C
- C74: value 2.2µF -> 2.2µF/25V; footprint Capacitor_SMD:C_0201_0603Metric -> Capacitor_SMD:C_0603_1608Metric
- C79: value 0.1µF -> 3.3nF/50V; footprint (none) -> Capacitor_SMD:C_0603_1608Metric
- C80: value Cac -> 100nF/50V; footprint (none) -> Capacitor_SMD:C_0603_1608Metric
- L5: footprint (none) -> Inductor_SMD:L_Bourns_SRR1260
- R31, R32, R33, R35, R36: footprint Resistor_SMD:R_01005_0402Metric -> Resistor_SMD:R_0603_1608Metric
- R34: value 51.1K -> 100K; footprint Resistor_SMD:R_0201_0603Metric -> Resistor_SMD:R_0603_1608Metric
Connections:
- net +12V: now also C81.1
- net +3.3V: now also C88.1
- net +36V: now also C75.2, C76.2
- net GND: now also C75.1, C76.1, C77.1, C81.2, C88.2
- net at L5.1, R34.1, U7.8 (SW): now also C78.2
- net at U7.7 (BST): now also C78.1
- net at U7.6 (VCC): now also C77.2
