File: Kicad Workspace/amplification.kicad_sch (KiCad schematic)
At the start: 49 parts, among them J5 L+, J6 L-, J7 R+, J8 R-, U5 TPA3255DDV

Commit message: fix: schematic corrections from the datasheet audit
Eight defects found by checking every pin of the six sheets against the
datasheets in Ressources/Datasheet.

MCU sheet:
- add R37/R41 (2.2K) I2C pull-ups on SDA/SCL, sized for the 400 kHz bus
- add R42 (2.2K) pull-up on PAIR_BT, SW2 had no defined idle level
- add C82/C83/C84 decoupling on the STM32 supply pins
- tie VREF+ to +3.3V, it was left unconnected so the ADC had no reference
- move the potentiometers and SW1 from +3.3VA to +3.3V, the analog rail is
  reserved for the audio path and the readings are ratiometric anyway

Amplification sheet:
- add C85 (10uF/25V) and C86 (0.1uF/16V) on the TPA3255 VDD, the 12V
  housekeeping rail had no local decoupling
Parts:
- added C85: 10µF/25V, Capacitor_SMD:C_0805_2012Metric, symbol Device:C
- added C86: 0.1µF/16V, Capacitor_SMD:C_0402_1005Metric, symbol Device:C
Connections:
- net +12V: now also C85.1, C86.1
- net GND: now also C85.2, C86.2

Commit message: feat: kicad alim stage clean up + TPA stage clean up
Parts:
- removed C59, C60, C61, C62: 10µF/50V, Capacitor_THT:C_Radial_D6.3mm_H11.0mm_P2.50mm, symbol Device:C
- added C60, C61, C62, C87: 10µF/50V, Capacitor_THT:CP_Radial_D6.3mm_P2.50mm, symbol Device:C_Polarized_US
- C33, C38, C39: value 1µF -> 1µF/25V; footprint Capacitor_SMD:C_0201_0603Metric -> Capacitor_SMD:C_0603_1608Metric
- C41, C42: footprint Capacitor_SMD:C_01005_0402Metric -> Capacitor_SMD:C_0603_1608Metric
- C43: value 33nF -> 33nF / 50V; footprint Capacitor_SMD:C_0201_0603Metric -> Capacitor_SMD:C_0603_1608Metric
- C44, C45, C46: value 33nF -> 33nF/50V; footprint Capacitor_SMD:C_0201_0603Metric -> Capacitor_SMD:C_0603_1608Metric
- C63, C64, C67, C68: footprint Capacitor_THT:C_Rect_L10.0mm_W4.0mm_P7.50mm_MKS4 -> Capacitor_SMD:C_1206_3216Metric
Connections:
- net IN_L+: now also C87.2
- net IN_L-: now also C60.2
- net IN_R+: now also C61.2
- net IN_R-: now also C62.2
- net at U5.16 (INPUT_C): now also C61.1
- net at U5.17 (INPUT_D): now also C62.1
- net at U5.5 (INPUT_A): now also C87.1
- net at U5.6 (INPUT_B): now also C60.1
